File: hardware/esp32_sync.sch (KiCad schematic (older format))
At the start: 107 parts, among them J11 USB_B_Micro, J12 Barrel_Jack, J2 Conn_01x02_Male, J21 GPIO, J22 I2S, J24 AUX0, J25 AUX1, J31 IDC SER, J32 SER1, J33 IDC SER, J34 SER2, J42 DS_3.3V, J43 DS0_EXT, J44 DS1_EXT, J45 DS2_EXT, J46 DS3_EXT, J51 AV, J52 AS0_EXT, J53 AS1_EXT, Q11 S8050, Q12 S8050, Q41 S8050, Q42 S8050, Q43 S8050, SW2 RESET, U1 CP2104, U11 SRV05-4, U13 AMS1117-3.3, U2 ESP32-WROOM-32D, U3 SP3232, U41 74AHC04, U42 74HC595, U43 74HC595, U45 TC4427, U46 TC4427, U51 DAC8562SDGSR, U52 NE5532, U53 NE5532

Commit message: Modified firmware for hardware, rev. 2 of PCB.
Parts:
- added CF13, CF3: 30PF/50V, Capacitor_SMD:C_0603_1608Metric, symbol Device:C
- added D44: GREEN, LED_SMD:LED_0603_1608Metric, symbol Device:LED
- added Q44: S8050, Package_TO_SOT_SMD:SOT-23, symbol Device:Q_NPN_BEC
- added RD47: 82, Resistor_SMD:R_0805_2012Metric, symbol Device:R
- added RD48: 4.7K, Resistor_SMD:R_0805_2012Metric, symbol Device:R
- added unit 3 of U41
- added unit 4 of U41
- added unit 5 of U41
- added unit 6 of U41
- J22: footprint Connector_PinHeader_2.54mm:PinHeader_1x04_P2.54mm_Vertical -> Connector_PinHeader_2.54mm:PinHeader_1x05_P2.54mm_Vertical; symbol Connector:Conn_01x04_Male -> Connector:Conn_01x05_Male
- renumbered C45A1 to C44, C45B1 to C45, C46A1 to C46, C46B1 to C47, CF0P1 to CF1, CF1P1 to CF11, CF1M1 to CF12, CF0M1 to CF2, RD41A1 to RD41, RD41B1 to RD42, RD42A1 to RD43, RD42B1 to RD44, RD43A1 to RD45, RD43B1 to RD46, R0_EXT1 to RO0, R1_EXT1 to RO1, R2_EXT1 to RO2, R3_EXT1 to RO3
Connections:
- net labels added: ~I2S_SCK
- wire segments 246 -> 257
Other:
- moved on the sheet: D42, Q42, RD43, RD44
